File: PCB/hackPad.kicad_sch (KiCad schematic)
At the start: 7 parts, among them SW1 SW_Push, SW2 SW_Push, SW3 SW_Push, SW4 SW_Push, U1 XIAO-RP2040-DIP

Commit message: Remade to add more changes to make the pad more unique
Parts:
- added SW5: RotaryEncoder_Switch, Rotary_Encoder:RotaryEncoder_Alps_EC11E-Switch_Vertical_H20mm, symbol Device:RotaryEncoder_Switch
Connections:
- net GND: now also SW5.C, SW5.S2
- net at U1.3 (GPIO28/ADC2/A2): now also SW5.B
- net at U1.4 (GPIO29/ADC3/A3): now also SW5.S1
- net at U1.6 (GPIO7/SCL): now also SW5.A
